Commit message: 完成go1训练和实机部署

File: resources/robots/go1/urdf/go1.urdf (robot description, URDF)
Before this commit: robot go1, 17 links, 16 joints
Links:
- added link imu, mass 0; collision box size=0.001 0.001 0.001; visual box size=0.001 0.001 0.001
- link FL_thigh: geometry collision box size=0.11 0.0245 0.034; visual mesh filename=../dae/thigh.dae scale=1 1 1
- link FR_thigh: geometry collision box size=0.11 0.0245 0.034; visual mesh filename=../dae/thigh_mirror.dae scale=1 1 1
- link RL_thigh: geometry collision box size=0.11 0.0245 0.034; visual mesh filename=../dae/thigh.dae scale=1 1 1
- link RR_thigh: geometry collision box size=0.11 0.0245 0.034; visual mesh filename=../dae/thigh_mirror.dae scale=1 1 1
- link base: geometry collision box size=0.3762 0.0935 0.114; visual mesh filename=../dae/trunk.dae scale=1 1 1
Joints:
- added joint imu_joint: type fixed, parent base, child imu, origin xyz=-0.01592 -0.06659 -0.00617 rpy=0 0 0, axis 0 0 0
- joint FL_hip_joint: origin xyz=0.1881 0.04675 0 rpy=0 -0 0 -> xyz=0.1881 0.04675 0 rpy=0 0 0
- joint FR_hip_joint: origin xyz=0.1881 -0.04675 0 rpy=0 -0 0 -> xyz=0.1881 -0.04675 0 rpy=0 0 0
- joint RL_hip_joint: origin xyz=-0.1881 0.04675 0 rpy=0 -0 0 -> xyz=-0.1881 0.04675 0 rpy=0 0 0
- joint RR_hip_joint: origin xyz=-0.1881 -0.04675 0 rpy=0 -0 0 -> xyz=-0.1881 -0.04675 0 rpy=0 0 0
